File: daisy/daisyEVI/daisyEVI.kicad_sch (KiCad schematic)
At the start: 0 parts

Commit message: Did Work on CAD; Now coding time
Parts:
- added A1: Electrosmith_Daisy_Seed_Rev4, Module:Electrosmith_Daisy_Seed, symbol MCU_Module:Electrosmith_Daisy_Seed_Rev4
- added SW1: RotaryEncoder_Switch, Rotary_Encoder:RotaryEncoder_Bourns_Horizontal_PEC09-2xxxF-Nxxxx, symbol Device:RotaryEncoder_Switch
- added U1: XGZP6847A005KPG33, symbol sensors:XGZP6847A005KPG33
